Commit message: Add: arm and bucket joint limit Changed: reward limit for episode

File: komodo2_description/urdf/komodo2.xacro (robot description, xacro)
@@ -561,5 +561,5 @@
     <axis
       xyz="-1 0 0" />
-    <limit effort="1000.0" lower="-0.5" upper="0.548" velocity="0.4"/>
+    <limit effort="1000.0" lower="-0.2" upper="0.32" velocity="0.1"/>
   </joint>
   <joint
@@ -575,5 +575,5 @@
     <axis
       xyz="-1 0 0" />
-    <limit effort="1000.0" lower="-0.5" upper="0.548" velocity="0.3"/>
+    <limit effort="1000.0" lower="-0.5" upper="0.548" velocity="0.05"/>
   </joint>
 </robot>

Commit message: Added control over reality komodo?

File: komodo2_description/urdf/komodo2.xacro (robot description, xacro)
@@ -561,5 +561,5 @@
     <axis
       xyz="-1 0 0" />
-    <limit effort="1000.0" lower="-0.2" upper="0.32" velocity="0.1"/>
+    <limit effort="290.0" lower="-0.2" upper="0.32" velocity="0.05"/>
   </joint>
   <joint
@@ -575,5 +575,5 @@
     <axis
       xyz="-1 0 0" />
-    <limit effort="1000.0" lower="-0.5" upper="0.548" velocity="0.05"/>
+    <limit effort="30.0" lower="-0.5" upper="0.548" velocity="0.05"/>
   </joint>
 </robot>

Commit message: fixed learning

File: komodo2_description/urdf/komodo2.xacro (robot description, xacro)
@@ -2,4 +2,5 @@
 <robot xmlns:xacro="http://www.ros.org/wiki/xacro" name="komodo2_robot" description="Komodo2 Robot">
 	<xacro:property name="M_PI" value="3.1415926535897931" />
+    <xacro:property name="Wheel_effort" value="0.05" />
       <link name="base_footprint"/>
  <joint name="base_footprint_joint" type="fixed">
@@ -16,12 +17,12 @@
         rpy="0 0 0" />
       <mass
-        value="200.0058" />
+        value="500.0058" />
       <inertia
-        ixx="0.80093"
+        ixx="80.0093"
         ixy="-0.37058"
         ixz="0.150841"
-        iyy="0.55849"
+        iyy="50.5849"
         iyz="-0.24895"
-        izz="1.02180" />
+        izz="10.2180" />
     </inertial>
     <visual>
@@ -102,5 +103,5 @@
       xyz="0 1 0" />
     <limit
-      effort="0.4"
+      effort="${Wheel_effort}"
       velocity="32.0" />
   </joint>
@@ -158,5 +159,5 @@
       xyz="0 1 0" />
     <limit
-      effort="0.4"
+      effort="${Wheel_effort}"
       velocity="32.0" />
   </joint>
@@ -214,5 +215,5 @@
       xyz="0 1 0" />
     <limit
-      effort="0.4"
+      effort="${Wheel_effort}"
       velocity="32.0" />
   </joint>
@@ -270,5 +271,5 @@
       xyz="0 1 0" />
     <limit
-      effort="0.4"
+      effort="${Wheel_effort}"
       velocity="32.0" />
   </joint>
@@ -561,5 +562,5 @@
     <axis
       xyz="-1 0 0" />
-    <limit effort="290.0" lower="-0.2" upper="0.32" velocity="0.05"/>
+    <limit effort="30.0" lower="-0.2" upper="0.32" velocity="0.07"/>
   </joint>
   <joint

Commit message: with force sensor smooth

File: komodo2_description/urdf/komodo2.xacro (robot description, xacro)
@@ -18,5 +18,14 @@
       <mass
         value="500.0058" />
-      <inertia
+      <!--mass
+        value="50.0058" /-->
+      <!--inertia
+        ixx="0.80093"
+        ixy="-0.37058"
+        ixz="0.150841"
+        iyy="0.55849"
+        iyz="-0.24895"
+        izz="1.02180" /-->
+    <inertia
         ixx="80.0093"
         ixy="-0.37058"
@@ -576,5 +585,5 @@
     <axis
       xyz="-1 0 0" />
-    <limit effort="30.0" lower="-0.5" upper="0.548" velocity="0.05"/>
+    <limit effort="20.0" lower="-0.5" upper="0.548" velocity="0.05"/>
   </joint>
 </robot>

File: komodo2_description/urdf/komodo2_gazebo.xacro (robot description, xacro)
@@ -97,4 +97,54 @@
                     </actuator>
                 </transmission>
+                <gazebo reference="bucket_joint">
+                    <provideFeedback>true</provideFeedback>
+                </gazebo>
+                <gazebo>
+                    <plugin name="ft_sensor" filename="libgazebo_ros_ft_sensor.so">
+                        <updateRate>80.0</updateRate>
+                        <topicName>bucket_torque_sensor</topicName>
+                        <jointName>bucket_joint</jointName>
+                    </plugin>
+                </gazebo>
+                <!--gazebo reference="bucket_joint">
+                <disableFixedJointLumping>true</disableFixedJointLumping>
+                <sensor name="FUCKING_SENSOR" type="force_torque">
+                  <force_torque>
+                    <frame>child</frame>
+                    <measure_direction>child_to_parent</measure_direction>
+                  </force_torque>
+                </sensor>
+              </gazebo-->
+              <!--gazebo>
+                  <plugin name="ft_sensor" filename="libgazebo_ros_ft_sensor.so">
+                      <updateRate>50.0</updateRate>
+                      <topicName>FUCKING_SENSOR</topicName>
+                      <jointName>bucket_joint</jointName>
+                  </plugin>
+              </gazebo-->
+                  <!--gazebo reference="bucket">
+                       <kp>1000000.0</kp>
+                        <kd>100.0</kd>
+                        <mu1>1.5</mu1>
+                        <mu2>1.5</mu2>
+                        <slip1>0.5</slip1>
+                        <slip2>0</slip2>
+                        <fdir1>1 0 0</fdir1>
+                        <maxVel>1.0</maxVel>
+                        <minDepth>0.00</minDepth>
+                    </gazebo-->
+                <!--gazebo reference="bucket">
+                      <sensor name="bucket_contact_sensor" type="contact">
+                        <always_on>true</always_on>
+                        <update_rate>30.0</update_rate>
+                        <contact>
+                          <collision>bucket_collision</collision>
+                        </contact>
+                        <plugin name="bucket_bumper" filename="libgazebo_ros_bumper.so">
+                          <bumperTopicName>bumper_contact_sensor_state</bumperTopicName>
+                          <frameName>bucket</frameName>
+                        </plugin>
+                      </sensor>
+                </gazebo-->
                 <xacro:transmission_arm joint_name="arm"/>
                 <xacro:transmission_arm joint_name="bucket"/>

Commit message: up to date , good learning

File: komodo2_description/urdf/komodo2.xacro (robot description, xacro)
@@ -488,5 +488,5 @@
       <mass
         value="1.6541" />
-      <!--inertia
+      <inertia
         ixx="0.020029"
         ixy="-3.1779E-16"
@@ -494,6 +494,6 @@
         iyy="0.0233"
         iyz="0.0034648"
-        izz="0.041275" /-->
-      <inertia ixx="1.0" ixy="0.0" ixz="0.0" iyy="1.0" iyz="0.0" izz="1.0" />
+        izz="0.041275" />
+      <!--inertia ixx="1.0" ixy="0.0" ixz="0.0" iyy="1.0" iyz="0.0" izz="1.0" /-->
     </inertial>
     <visual>
@@ -525,5 +525,5 @@
       <mass
         value="0.74403" />
-      <!--inertia
+      <inertia
         ixx="0.00060709"
         ixy="1.575E-16"
@@ -531,6 +531,6 @@
         iyy="0.0060723"
         iyz="-4.2694E-06"
-        izz="0.0066375" /-->
-      <inertia ixx="1.0" ixy="0.0" ixz="0.0" iyy="1.0" iyz="0.0" izz="1.0" />
+        izz="0.0066375" />
+      <!--inertia ixx="1.0" ixy="0.0" ixz="0.0" iyy="1.0" iyz="0.0" izz="1.0" /-->
     </inertial>
     <visual>
@@ -571,5 +571,6 @@
     <axis
       xyz="-1 0 0" />
-    <limit effort="30.0" lower="-0.2" upper="0.32" velocity="0.07"/>
+    <limit effort="30.0" lower="-0.2" upper="0.32" velocity="0.2"/>
+    <dynamics damping="40" friction="0.1"/>
   </joint>
   <joint
@@ -585,5 +586,6 @@
     <axis
       xyz="-1 0 0" />
-    <limit effort="20.0" lower="-0.5" upper="0.548" velocity="0.05"/>
+    <dynamics damping="1" friction="0.0"/>
+    <limit effort="7.0" lower="-0.5" upper="0.548" velocity="0.01"/>
   </joint>
 </robot>

Commit message: changed limits

File: komodo2_description/urdf/komodo2.xacro (robot description, xacro)
@@ -571,5 +571,5 @@
     <axis
       xyz="-1 0 0" />
-    <limit effort="30.0" lower="-0.2" upper="0.32" velocity="0.2"/>
+    <limit effort="30.0" lower="-0.1" upper="0.32" velocity="0.2"/>
     <dynamics damping="40" friction="0.1"/>
   </joint>
@@ -587,5 +587,5 @@
       xyz="-1 0 0" />
     <dynamics damping="1" friction="0.0"/>
-    <limit effort="7.0" lower="-0.5" upper="0.548" velocity="0.01"/>
+    <limit effort="7.0" lower="-0.5" upper="0.9" velocity="0.01"/>
   </joint>
 </robot>

Commit message: added new state

File: komodo2_description/urdf/komodo2.xacro (robot description, xacro)
@@ -14,24 +14,16 @@
     <inertial>
       <origin
-        xyz="0.0030152 0.00057861 0.0749"
-        rpy="0 0 0" />
-      <mass
-        value="500.0058" />
-      <!--mass
-        value="50.0058" /-->
-      <!--inertia
-        ixx="0.80093"
-        ixy="-0.37058"
-        ixz="0.150841"
-        iyy="0.55849"
-        iyz="-0.24895"
-        izz="1.02180" /-->
-    <inertia
-        ixx="80.0093"
-        ixy="-0.37058"
-        ixz="0.150841"
-        iyy="50.5849"
-        iyz="-0.24895"
-        izz="10.2180" />
+        xyz="0.0 0.0 0.0749"
+        rpy="0 0 0" />
+      <mass
+        value="40.0058" />
+      <!--inertia 20
+        ixx="0.1927" ixy="0.0" ixz="0.0"
+        iyy="0.5366" iyz="0.0"
+        izz="0.5959"/-->
+      <inertia
+        ixx="0.385" ixy="0.0" ixz="0.0"
+        iyy="1.072" iyz="0.0"
+        izz="1.1919"/>
     </inertial>
     <visual>
@@ -51,9 +43,10 @@
     <collision>
       <origin
-        xyz="0 0 0"
-        rpy="0 0 0" />
-      <geometry>
-        <mesh
-          filename="package://komodo2_description/mesh/base.STL" />
+        xyz="0 0 0.0749"
+        rpy="0 0 0" />
+      <geometry>
+        <!--mesh
+          filename="package://komodo2_description/mesh/base.STL" /-->
+        <box size="0.531 0.275 0.2"/>
       </geometry>
     </collision>
@@ -311,7 +304,7 @@
     <axis
       xyz="0 0 0" />
-    <limit
+    <!--limit
       effort="0.4"
-      velocity="32.0" />
+      velocity="32.0" /-->
   </joint>
   <link
@@ -453,10 +446,10 @@
         value="1.6502" />
       <inertia
-        ixx="0.5"
+        ixx="0.05"
         ixy="0"
         ixz="0"
-        iyy="0.5"
+        iyy="0.05"
         iyz="0"
-        izz="0.5" />
+        izz="0.05" />
     </inertial>
     <visual>
@@ -571,5 +564,5 @@
     <axis
       xyz="-1 0 0" />
-    <limit effort="30.0" lower="-0.1" upper="0.32" velocity="0.2"/>
+    <limit effort="100.0" lower="-0.1" upper="0.32" velocity="0.2"/>
     <dynamics damping="40" friction="0.1"/>
   </joint>
@@ -586,6 +579,6 @@
     <axis
       xyz="-1 0 0" />
-    <dynamics damping="1" friction="0.0"/>
-    <limit effort="7.0" lower="-0.5" upper="0.9" velocity="0.01"/>
+    <dynamics damping="2" friction="0.9"/>
+    <limit effort="30.0" lower="-0.5" upper="0.9" velocity="0.01"/>
   </joint>
 </robot>

File: komodo2_description/urdf/komodo2_gazebo.xacro (robot description, xacro)
@@ -102,5 +102,5 @@
                 <gazebo>
                     <plugin name="ft_sensor" filename="libgazebo_ros_ft_sensor.so">
-                        <updateRate>80.0</updateRate>
+                        <updateRate>10.0</updateRate>
                         <topicName>bucket_torque_sensor</topicName>
                         <jointName>bucket_joint</jointName>
